File: esp32.kicad_sch (KiCad schematic)
At the start: 11 parts, among them J201 USB_B_Micro, J202 JTAG, U201 USBLC6-2SC6, U202 ESP32-S3-WROOM-1

Commit message: Rework order information
Signed-off-by: Benedikt Spranger <b.spranger@linutronix.de>
Parts:
- D201: Long Description (none) -> -40℃~+85℃ 0.6mA 1.95mm 120° 1kHz 2000V 3.5mm 3.7V~5.5V 3.7m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; MF (none) -> OPSCO Optoelectronics; MP (none) -> SK6812MINI-HS; Source (none) -> JLCPCB; SupplLink (none) -> https://jlcpcb.com/partdetail/OPSCOOptoelectronics-SK6812MI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; lcsc# (none) -> C2922787
- FB201: Long Description (none) -> -55℃~+125℃ 1 120Ω@100MHz 2A 50mΩ ±25% 0603 Ferrite Beads RO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; MF (none) -> Murata Electronics; MP (none) -> BLM18PG121SN1D; Source (none) -> JLCPCB; SupplLink (none) -> https://jlcpcb.com/partdetail/MurataElectronics-BLM18PG121S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; lcsc# (none) -> C14709
- J201: Long Description (none) -> -30℃~+80℃ 1 5P Female Micro-B Surface Mount, Right Angle US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; MF (none) -> Amphenol ICC; MP (none) -> 10103594-0001LF; Source (none) -> JLCPCB; SupplLink (none) -> https://jlcpcb.com/partdetail/AmphenolICC-101035940001LF/C4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; lcsc# (none) -> C428495
- J202: MF (none) -> Tag Connect; MP (none) -> TC2050-IDC-FP; Source (none) -> ---
- JP201, JP202, JP204, JP205: MP (none) -> N/A; Source (none) -> ---
- JP203: Long Description (none) -> Connector: pin strips; pin header; male; PIN: 3; THT; strai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; MF (none) -> CONNFLY; MP (none) -> DS1021-1*3SF11-B; Source (none) -> TME; SupplLink (none) -> https://www.tme.eu/de/en/details/zl201-03g/pin-headers/conn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; tme# (none) -> ZL201-03G
- U201: Long Description (none) -> 0.8pF 100nA 150W@8/20us 15V 2 5V 6A@8/20us 6V ESD SOT-23-6 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; MF (none) -> UMW(Youtai Semiconductor Co., Ltd.); MP (none) -> USBLC6-2SC6; Source (none) -> JLCPCB; SupplLink (none) -> https://jlcpcb.com/partdetail/2790619-USBLC62SC6/C2687116; lcsc# (none) -> C2687116
- U202: Long Description (none) -> SMD,19.2x18mm WiFi Modules ROHS; MF (none) -> Espressif Systems; MP (none) -> ESP32-S3-WROOM-1U-N16R8; Source (none) -> JLCPCB; SupplLink (none) -> https://jlcpcb.com/partdetail/3522416-ESP32_S3_WROOM_1UN16R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; lcsc# (none) -> C3013946
