File: esp32.kicad_sch (KiCad schematic)
At the start: 11 parts, among them J201 USB_B_Micro, J202 JTAG, U201 USBLC6-2SC6, U202 ESP32-S3-WROOM-1

Commit message: Fix SK6812 footprint mess
Signed-off-by: Benedikt Spranger <b.spranger@linutronix.de>
Parts:
- D201: value SK6812MINI -> SK6812MINI-HS-012; footprint LED_SMD:LED_SK6812MINI_PLCC4_3.5x3.5mm_P1.75mm -> LED_SMD:LED_WS2812B-Mini_PLCC4_3.5x3.5mm; symbol LED:SK6812MINI -> sk6812mini:SK6812MINI-HS-012
Connections:
- net +3V3: now also D201.3 (VDD); no longer D201.4 (VDD)
- net GNDD: now also D201.1 (VSS); no longer D201.2 (VSS)
- net at U202.31 (GPIO38/FSPIWP/SUBSPIWP): now also D201.2 (DIN); no longer D201.3 (DIN)
Changed lines of the file:
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@@
 	)
 	(symbol
-		(lib_id "LED:SK6812MINI")
+		(lib_id "sk6812mini:SK6812MINI-HS-012")
 		(at 228.6 106.68 0)
 		(unit 1)
@@
 		(on_board yes)
 		(dnp no)
-		(fields_autoplaced yes)
 		(property "Reference" "D201"
-			(at 241.3 100.2598 0)
+			(at 236.474 100.33 0)
 			(effects
 				(font
@@
 			)
 		)
-		(property "Value" "SK6812MINI"
-			(at 241.3 102.7998 0)
+		(property "Value" "SK6812MINI-HS-012"
+			(at 244.348 102.362 0)
 			(effects
 				(font
@@
 			)
 		)
-		(property "Footprint" "LED_SMD:LED_SK6812MINI_PLCC4_3.5x3.5mm_P1.75mm"
+		(property "Footprint" "LED_SMD:LED_WS2812B-Mini_PLCC4_3.5x3.5mm"
 			(at 229.87 114.3 0)
 			(effects
@@
 			)
 		)
-		(property "Datasheet" "https://cdn-shop.adafruit.com/product-files/2686/SK6812MINI_REV.01-1-2.pdf"
+		(property "Datasheet" "https://jlcpcb.com/api/file/downloadByFileSystemAccessId/8588920813789581312"
 			(at 231.14 116.205 0)
 			(effects
