File: com4bbb.kicad_sch (KiCad schematic)
At the start: 50 parts, among them J101 PWR, J102 RS485, P8 BeagleBone_Black_Header, P9 BeagleBone_Black_Header, SW101 Reset, SW102 PWR, U101 WPMDH1100xx1S, U102 AT24C512C-SSHD-T, U103 SP3485EN, U104 ESP32-WROOM-32U

Commit message: Update to ESP32-S3-WROOM-1U
Signed-off-by: Benedikt Spranger <bene@eurovibes.org>
Parts:
- removed D114: 1N4004, Diode_THT:D_DO-41_SOD81_P10.16mm_Horizontal, symbol Diode:1N4004
- removed JP101: TX, Jumper:SolderJumper-3_P1.3mm_Open_RoundedPad1.0x1.5mm, symbol Jumper:Jumper_3_Open
- removed JP102: RX, Jumper:SolderJumper-3_P1.3mm_Open_RoundedPad1.0x1.5mm, symbol Jumper:Jumper_3_Open
- removed JP103: VSPIQ, Jumper:SolderJumper-3_P1.3mm_Open_RoundedPad1.0x1.5mm, symbol Jumper:Jumper_3_Open
- removed JP104: VSPID, Jumper:SolderJumper-3_P1.3mm_Open_RoundedPad1.0x1.5mm, symbol Jumper:Jumper_3_Open
- removed U104: ESP32-WROOM-32U, RF_Module:ESP32-WROOM-32U, symbol RF_Module:ESP32-WROOM-32U
- added D114: MRA4004T3G, Diode_SMD:D_SMA, symbol Diode:MRA4004T3G
- C101: LCSC C1525 -> (none); Long Description (none) -> 100nF 16V X7R ±10% 0402 Multilayer Ceramic Capacitors MLCC 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; MF (none) -> Samsung Electro-Mechanics; MP (none) -> CL05B104KO5NNNC; ManuPart# CL05B104KO5NNNC -> (none); Manufacture Samsung Electro-Mechanics -> (none); Source (none) -> JLCPCB; SupplLink (none) -> https://jlcpcb.com/partdetail/1877-CL05B104KO5NNNC/C1525; lcsc# (none) -> C1525
- D101: renamed from D113; LCSC C2286 -> (none); MF (none) -> Hubei KENTO Elec; MP (none) -> KT-0603R; ManuPart# KT-0603R -> (none); Manufacture Hubei KENTO Elec -> (none); Source (none) -> JLCPCB; lcsc# (none) -> C2286
- D102: renamed from D101; LCSC C2286 -> (none); MF (none) -> Hubei KENTO Elec; MP (none) -> KT-0603R; ManuPart# KT-0603R -> (none); Manufacture Hubei KENTO Elec -> (none); Source (none) -> JLCPCB; lcsc# (none) -> C2286
- D103: renamed from D102; LCSC C2286 -> (none); MF (none) -> Hubei KENTO Elec; MP (none) -> KT-0603R; ManuPart# KT-0603R -> (none); Manufacture Hubei KENTO Elec -> (none); Source (none) -> JLCPCB; lcsc# (none) -> C2286
- D104: renamed from D103; LCSC C2286 -> (none); MF (none) -> Hubei KENTO Elec; MP (none) -> KT-0603R; ManuPart# KT-0603R -> (none); Manufacture Hubei KENTO Elec -> (none); Source (none) -> JLCPCB; lcsc# (none) -> C2286
- D105: renamed from D104; LCSC C2286 -> (none); MF (none) -> Hubei KENTO Elec; MP (none) -> KT-0603R; ManuPart# KT-0603R -> (none); Manufacture Hubei KENTO Elec -> (none); Source (none) -> JLCPCB; lcsc# (none) -> C2286
- D106: renamed from D105; LCSC C2286 -> (none); MF (none) -> Hubei KENTO Elec; MP (none) -> KT-0603R; ManuPart# KT-0603R -> (none); Manufacture Hubei KENTO Elec -> (none); Source (none) -> JLCPCB; lcsc# (none) -> C2286
- D107: renamed from D106; LCSC C2286 -> (none); MF (none) -> Hubei KENTO Elec; MP (none) -> KT-0603R; ManuPart# KT-0603R -> (none); Manufacture Hubei KENTO Elec -> (none); Source (none) -> JLCPCB; lcsc# (none) -> C2286
- D108: renamed from D107; LCSC C2286 -> (none); MF (none) -> Hubei KENTO Elec; MP (none) -> KT-0603R; ManuPart# KT-0603R -> (none); Manufacture Hubei KENTO Elec -> (none); Source (none) -> JLCPCB; lcsc# (none) -> C2286
- D109: renamed from D108; LCSC C2286 -> (none); MF (none) -> Hubei KENTO Elec; MP (none) -> KT-0603R; ManuPart# KT-0603R -> (none); Manufacture Hubei KENTO Elec -> (none); Source (none) -> JLCPCB; lcsc# (none) -> C2286
- D110: renamed from D109; LCSC C2286 -> (none); MF (none) -> Hubei KENTO Elec; MP (none) -> KT-0603R; ManuPart# KT-0603R -> (none); Manufacture Hubei KENTO Elec -> (none); Source (none) -> JLCPCB; lcsc# (none) -> C2286
- D111: renamed from D110; LCSC C2286 -> (none); MF (none) -> Hubei KENTO Elec; MP (none) -> KT-0603R; ManuPart# KT-0603R -> (none); Manufacture Hubei KENTO Elec -> (none); Source (none) -> JLCPCB; lcsc# (none) -> C2286
- D112: renamed from D111; LCSC C2286 -> (none); MF (none) -> Hubei KENTO Elec; MP (none) -> KT-0603R; ManuPart# KT-0603R -> (none); Manufacture Hubei KENTO Elec -> (none); Source (none) -> JLCPCB; lcsc# (none) -> C2286
- D113: renamed from D112; LCSC C2286 -> (none); MF (none) -> Hubei KENTO Elec; MP (none) -> KT-0603R; ManuPart# KT-0603R -> (none); Manufacture Hubei KENTO Elec -> (none); Source (none) -> JLCPCB; lcsc# (none) -> C2286
- J101: renamed from J102; footprint TerminalBlock_WAGO:TerminalBlock_WAGO_236-102_1x02_P5.00mm_45Degree -> TerminalBlock_WAGO:TerminalBlock_WAGO_236-402_1x02_P5.00mm_45Degree; assemble y -> n
- J102: renamed from J101; footprint TerminalBlock_Phoenix:TerminalBlock_Phoenix_MPT-0,5-2-2.54_1x02_P2.54mm_Horizontal -> TerminalBlock_WAGO:TerminalBlock_WAGO_236-402_1x02_P5.00mm_45Degree; assemble (none) -> n
- R101: renamed from R105; LCSC C11702 -> (none); MF (none) -> UNI-ROYAL(Uniroyal Elec); MP (none) -> 0402WGF1001TCE; ManuPart# 0402WGF1001TCE -> (none); Manufacture UNI-ROYAL(Uniroyal Elec) -> (none); Source (none) -> JLCPCB; lcsc# (none) -> C11702
- R102: renamed from R106; LCSC C11702 -> (none); MF (none) -> UNI-ROYAL(Uniroyal Elec); MP (none) -> 0402WGF1001TCE; ManuPart# 0402WGF1001TCE -> (none); Manufacture UNI-ROYAL(Uniroyal Elec) -> (none); Source (none) -> JLCPCB; lcsc# (none) -> C11702
- R103: renamed from R107; LCSC C11702 -> (none); MF (none) -> UNI-ROYAL(Uniroyal Elec); MP (none) -> 0402WGF1001TCE; ManuPart# 0402WGF1001TCE -> (none); Manufacture UNI-ROYAL(Uniroyal Elec) -> (none); Source (none) -> JLCPCB; lcsc# (none) -> C11702
- R104: renamed from R108; LCSC C11702 -> (none); MF (none) -> UNI-ROYAL(Uniroyal Elec); MP (none) -> 0402WGF1001TCE; ManuPart# 0402WGF1001TCE -> (none); Manufacture UNI-ROYAL(Uniroyal Elec) -> (none); Source (none) -> JLCPCB; lcsc# (none) -> C11702
- R105: renamed from R109; LCSC C11702 -> (none); MF (none) -> UNI-ROYAL(Uniroyal Elec); MP (none) -> 0402WGF1001TCE; ManuPart# 0402WGF1001TCE -> (none); Manufacture UNI-ROYAL(Uniroyal Elec) -> (none); Source (none) -> JLCPCB; lcsc# (none) -> C11702
- R106: renamed from R110; LCSC C11702 -> (none); MF (none) -> UNI-ROYAL(Uniroyal Elec); MP (none) -> 0402WGF1001TCE; ManuPart# 0402WGF1001TCE -> (none); Manufacture UNI-ROYAL(Uniroyal Elec) -> (none); Source (none) -> JLCPCB; lcsc# (none) -> C11702
- R107: renamed from R111; LCSC C11702 -> (none); MF (none) -> UNI-ROYAL(Uniroyal Elec); MP (none) -> 0402WGF1001TCE; ManuPart# 0402WGF1001TCE -> (none); Manufacture UNI-ROYAL(Uniroyal Elec) -> (none); Source (none) -> JLCPCB; lcsc# (none) -> C11702
- R108: renamed from R112; LCSC C11702 -> (none); MF (none) -> UNI-ROYAL(Uniroyal Elec); MP (none) -> 0402WGF1001TCE; ManuPart# 0402WGF1001TCE -> (none); Manufacture UNI-ROYAL(Uniroyal Elec) -> (none); Source (none) -> JLCPCB; lcsc# (none) -> C11702
- R109: renamed from R113; LCSC C11702 -> (none); MF (none) -> UNI-ROYAL(Uniroyal Elec); MP (none) -> 0402WGF1001TCE; ManuPart# 0402WGF1001TCE -> (none); Manufacture UNI-ROYAL(Uniroyal Elec) -> (none); Source (none) -> JLCPCB; lcsc# (none) -> C11702
- R110: renamed from R114; LCSC C11702 -> (none); MF (none) -> UNI-ROYAL(Uniroyal Elec); MP (none) -> 0402WGF1001TCE; ManuPart# 0402WGF1001TCE -> (none); Manufacture UNI-ROYAL(Uniroyal Elec) -> (none); Source (none) -> JLCPCB; lcsc# (none) -> C11702
- R111: renamed from R115; LCSC C11702 -> (none); MF (none) -> UNI-ROYAL(Uniroyal Elec); MP (none) -> 0402WGF1001TCE; ManuPart# 0402WGF1001TCE -> (none); Manufacture UNI-ROYAL(Uniroyal Elec) -> (none); Source (none) -> JLCPCB; lcsc# (none) -> C11702
- R112: renamed from R116; LCSC C11702 -> (none); MF (none) -> UNI-ROYAL(Uniroyal Elec); MP (none) -> 0402WGF1001TCE; ManuPart# 0402WGF1001TCE -> (none); Manufacture UNI-ROYAL(Uniroyal Elec) -> (none); Source (none) -> JLCPCB; lcsc# (none) -> C11702
- R113: renamed from R117; LCSC C11702 -> (none); MF (none) -> UNI-ROYAL(Uniroyal Elec); MP (none) -> 0402WGF1001TCE; ManuPart# 0402WGF1001TCE -> (none); Manufacture UNI-ROYAL(Uniroyal Elec) -> (none); Source (none) -> JLCPCB; lcsc# (none) -> C11702
- R114: renamed from R101; LCSC C11702 -> (none); MF (none) -> UNI-ROYAL(Uniroyal Elec); MP (none) -> 0402WGF1001TCE; ManuPart# 0402WGF1001TCE -> (none); Manufacture UNI-ROYAL(Uniroyal Elec) -> (none); Source (none) -> JLCPCB; lcsc# (none) -> C11702
- R115: renamed from R102; LCSC C11702 -> (none); MF (none) -> UNI-ROYAL(Uniroyal Elec); MP (none) -> 0402WGF1001TCE; ManuPart# 0402WGF1001TCE -> (none); Manufacture UNI-ROYAL(Uniroyal Elec) -> (none); Source (none) -> JLCPCB; lcsc# (none) -> C11702
- R116: renamed from R103; LCSC C11702 -> (none); MF (none) -> UNI-ROYAL(Uniroyal Elec); MP (none) -> 0402WGF1001TCE; ManuPart# 0402WGF1001TCE -> (none); Manufacture UNI-ROYAL(Uniroyal Elec) -> (none); Source (none) -> JLCPCB; lcsc# (none) -> C11702
- R117: renamed from R104; LCSC C11702 -> (none); MF (none) -> UNI-ROYAL(Uniroyal Elec); MP (none) -> 0402WGF1001TCE; ManuPart# 0402WGF1001TCE -> (none); Manufacture UNI-ROYAL(Uniroyal Elec) -> (none); Source (none) -> JLCPCB; lcsc# (none) -> C11702
- U101: renamed from U103; LCSC C8963 -> (none); MF (none) -> MaxLinear; MP (none) -> SP3485EN-L/TR; ManuPart# SP3485EN-L/TR -> (none); Manufacture MaxLinear -> (none); Source (none) -> JLCPCB; lcsc# (none) -> C8963
- U102: renamed from U101; assemble (none) -> n
- U103: renamed from U102; LCSC C6482 -> (none); MF (none) -> Microchip Tech; MP (none) -> AT24C256C-SSHL-T; ManuPart# AT24C256C-SSHL-T -> (none); Manufacture Microchip Tech -> (none); Source (none) -> JLCPCB; lcsc# (none) -> C6482
- renumbered JP105 to JP101, JP106 to JP102, JP107 to JP103, JP108 to JP104
Connections:
- net at R101.1: now also D101.1 (K); no longer D102.1 (K)
- net at D103.1 (K): now also R103.1; no longer R102.1
- net at D104.1 (K): now also R104.1; no longer R103.1
- net at D105.1 (K): now also R105.1; no longer R104.1
- net at D106.1 (K): now also R106.1; no longer R105.1
- net at D107.1 (K): now also R107.1; no longer R106.1
- net at D108.1 (K): now also R108.1; no longer R107.1
- net at D109.1 (K): now also R109.1; no longer R108.1
- net at D110.1 (K): now also R110.1; no longer R109.1
- net at D111.1 (K): now also R111.1; no longer R110.1
- net at D112.1 (K): now also R112.1; no longer R111.1
- net at D113.1 (K): now also R113.1; no longer R112.1
- net at J102.2 (Pin_2): now also D114.2 (A)
- net at U102.1 (Vin): now also D114.1 (K)
- new net: D102.1 (K), R102.1
- no-connect marks 69 -> 46
Other:
- added sheet ESP32 (esp32.kicad_sch)
- note removed: "internal use do not connect"
- moved on the sheet: D101, D102, D103, D104, D105, D106, D107, D108, D109, D110, D111, D112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

Commit message: Rework order information
Signed-off-by: Benedikt Spranger <b.spranger@linutronix.de>
Parts:
- D101, D102, D103, D104, D105, D106, D107, D108, D109, D110, D111, D112, D113: Long Description (none) -> -40℃~+85℃ 120° 2.4V 20mA 300mcd 40mW 615nm~630nm 645nm Red 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; SupplLink (none) -> https://jlcpcb.com/partdetail/Hubei_KENTOElec-KT0603R/C2286
- J101, J102: Long Description (none) -> 2 Position Wire to Board Terminal Block 45° (135°) Angle wi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; MF (none) -> WAGO Corporation; MP (none) -> 236-402; Source (none) -> Digikey; digikey# (none) -> 2946-236-402-ND
- JP101, JP102, JP103, JP104: MP (none) -> N/A; Source (none) -> ---
- P8, P9: MF (none) -> SAMTEC; MP (none) -> TSW-123-07-T-D; Source (none) -> TME; SupplLink (none) -> https://www.tme.eu/de/en/details/tsw-123-07-t-d/pin-headers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; tme# (none) -> TSW-123-07-T-D
- R101, R102, R103, R104, R105, R106, R107, R108, R109, R110, R111, R112, R113, R114, R115, R116, R117: Long Description (none) -> -55℃~+155℃ 1kΩ 50V 62.5mW Thick Film Resistor ±1% ±100ppm/℃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; SupplLink (none) -> https://jlcpcb.com/partdetail/12256-0402WGF1001TCE/C11702
- SW101, SW102: Long Description (none) -> Microswitch TACT; SPST-NO; Pos: 2; 0.05A/12VDC; THT; none; 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; MF (none) -> NINIGI; MP (none) -> TACT-64N-F; Source (none) -> TME; SupplLink (none) -> https://www.tme.eu/de/en/details/tact-64n-f/microswitches-t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; tme# (none) -> TACT-64N-F
- U101: Long Description (none) -> -40℃~+85℃ 1 1 10Mbps 2mA 3.3V 32 Half-Duplex Transceiver SO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; SupplLink (none) -> https://jlcpcb.com/partdetail/MaxLinear-SP3485EN_LTR/C8963
- U102: value WPMDH1100xx1S -> R-78K5.0-0.5; Long Description (none) -> Converter: DC/DC; Uin: 6.5÷36VDC; Uout: 5VDC; Iout: 500mA; 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; MF (none) -> RECOM; MP (none) -> R-78K5.0-0.5; Source (none) -> TME; SupplLink (none) -> https://www.tme.eu/de/en/details/r-78k5.0-0.5/dc-dc-convert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; tme# (none) -> R-78K5.0-0.5
- U103: Long Description (none) -> -40℃~+85℃ 1,000,000 Cycles 1.7V~5.5V 1MHz 256Kbit 40 Years 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; SupplLink (none) -> https://jlcpcb.com/partdetail/MicrochipTech-AT24C256C_SSHLT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

Commit message: Add RTC and secure memory
Signed-off-by: Benedikt Spranger <bene@eurovibes.org>
Parts:
- added C102: 100n, Capacitor_SMD:C_0402_1005Metric, symbol Device:C
- added C103, C104: 1F, Capacitor_THT:CP_Radial_D8.0mm_P3.50mm, symbol Device:C_Polarized
- added D115: 1N5819WS, Diode_SMD:D_SOD-323, symbol Diode:1N5819WS
- added R118: 15, Resistor_SMD:R_0805_2012Metric, symbol Device:R
- added TP101: 32kHz, TestPoint:TestPoint_Pad_1.0x1.0mm, symbol Connector:TestPoint
- added U104: ATECC608A-MAHDA, Package_DFN_QFN:DFN-8-1EP_3x2mm_P0.5mm_EP1.3x1.5mm, symbol Security:ATECC608A-MAHDA
- added U105: DS3231MZ, Package_SO:SOIC-8_3.9x4.9mm_P1.27mm, symbol Timer_RTC:DS3231MZ
Connections:
- net +3V3: now also D115.2 (A), U104.8 (VCC), U105.6 (VBAT)
- net GNDD: now also C102.2, C103.2, C104.2, U104.4 (GND), U104.9 (EP), U105.5 (GND)
- net SCL: now also U104.6 (SCL), U105.8 (SCL)
- net SDA: now also U104.5 (SDA), U105.7 (SDA)
- net SYS_RESETN: now also U105.4 (~{RST})
- net RTC_INT: now reaches P9.14 (Pin_14)
- net RTC_INT: now also U105.3 (~{INT}/SQW)
- new net: D115.1 (K), R118.1
- new net: TP101.1, U105.1 (32KHZ)
- new net Vbat: C102.1, C103.1, C104.1, R118.2, U105.2 (VCC)
- no-connect marks 46 -> 45

Commit message: Add DCF77 clock input
Signed-off-by: Benedikt Spranger <b.spranger@linutronix.de>
Parts:
- added J103: DCF77, Connector_PinHeader_2.54mm:PinHeader_1x02_P2.54mm_Vertical, symbol Connector_Generic:Conn_01x02
Connections:
- net GNDD: now also J103.2 (Pin_2)
- net DCF77: now reaches P9.16 (Pin_16)
- net DCF77: now also J103.1 (Pin_1)
- no-connect marks 45 -> 44
Changed lines of the file:
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@@
 	)
 	(no_connect
-		(at 63.5 46.99)
-	)
-	(no_connect
 		(at 119.38 64.77)
 	)
@@
 	(wire
 		(pts
+			(xy 63.5 46.99) (xy 66.04 46.99)
+		)
+		(stroke
+			(width 0)
+			(type default)
+		)
+	)
+	(wire
+		(pts
 			(xy 25.4 152.4) (xy 25.4 154.94)
 		)
@@
 	(wire
 		(pts
+			(xy 165.1 76.2) (xy 167.64 76.2)
+		)
+		(stroke
+			(width 0)
+			(type default)
+		)
+	)
+	(wire
+		(pts
 			(xy 213.36 106.68) (xy 215.9 106.68)
 		)
@@
 	(wire
 		(pts
+			(xy 165.1 78.74) (xy 165.1 81.28)
+		)
+		(stroke
+			(width 0)
+			(type default)
+		)
+	)
+	(wire
+		(pts
 			(xy 152.4 111.76) (xy 152.4 114.3)
 		)
@@
 	(wire
 		(pts
+			(xy 167.64 78.74) (xy 165.1 78.74)
+		)
+		(stroke
+			(width 0)
+			(type default)
+		)
+	)
+	(wire
+		(pts
 			(xy 144.78 172.72) (xy 147.32 172.72)
 		)
@@
 		)
 	)
+	(label "DCF77"
+		(at 66.04 46.99 0)
+		(effects
+			(font
+				(size 1.27 1.27)
+			)
+			(justify left bottom)
+		)
+	)
 	(label "LED3"
 		(at 134.62 39.37 0)
@@
 		)
 	)
+	(label "DCF77"
+		(at 165.1 76.2 180)
+		(effects
+			(font
+				(size 1.27 1.27)
+			)
+			(justify right bottom)
+		)
+	)
 	(label "LED8"
 		(at 215.9 152.4 270)
@@
 	(symbol
 		(lib_id "power:GNDD")
+		(at 165.1 81.28 0)
+		(unit 1)
+		(exclude_from_sim no)
+		(in_bom yes)
+		(on_board yes)
+		(dnp no)
+		(property "Reference" "#PWR0154"
+			(at 165.1 87.63 0)
+			(effects
+				(font
+					(size 1.27 1.27)
+				)
+				(hide yes)
+			)
+		)
+		(property "Value" "GNDD"
+			(at 165.1 85.09 0)
+			(effects
+				(font
+					(size 1.27 1.27)
+				)
+			)
+		)
+		(property "Footprint" ""
+			(at 165.1 81.28 0)
+			(effects
+				(font
+					(size 1.524 1.524)
+				)
+				(hide yes)
+			)
+		)
+		(property "Datasheet" ""
+			(at 165.1 81.28 0)
+			(effects
+				(font
+					(size 1.524 1.524)
+				)
+				(hide yes)
+			)
+		)
+		(property "Description" "Power symbol creates a global label with name \"GNDD\" , digital ground"
+			(at 165.1 81.28 0)
+			(effects
+				(font
+					(size 1.27 1.27)
+				)
+				(hide yes)
+			)
+		)
+		(pin "1"
+		)
+		(instances
+			(project "com4bbb"
+				(path "/bfd666b6-a268-42c4-a4e5-052a7c5965f6"
+					(reference "#PWR0154")
+					(unit 1)
+				)
+			)
+		)
+	)
+	(symbol
+		(lib_id "power:GNDD")
 		(at 241.3 104.14 0)
 		(unit 1)
@@
 					(unit 1)
 				)
+			)
+		)
+	)
+	(symbol
+		(lib_id "Connector_Generic:Conn_01x02")
+		(at 172.72 76.2 0)
+		(unit 1)
+		(exclude_from_sim no)
+		(in_bom yes)
+		(on_board yes)
+		(dnp no)
+		(fields_autoplaced yes)
+		(property "Reference" "J103"
+			(at 175.26 76.1999 0)
+			(effects
+				(font
+					(size 1.27 1.27)
+				)
+				(justify left)
+			)
+		)
+		(property "Value" "DCF77"
+			(at 175.26 78.7399 0)
+			(effects
+				(font
+					(size 1.27 1.27)
+				)
+				(justify left)
+			)
+		)
+		(property "Footprint" "Connector_PinHeader_2.54mm:PinHeader_1x02_P2.54mm_Vertical"
+			(at 172.72 76.2 0)
+			(effects
+				(font
+					(size 1.27 1.27)
+				)
+				(hide yes)
+			)
+		)
+		(property "Datasheet" "~"
+			(at 172.72 76.2 0)
+			(effects
+				(font
+					(size 1.27 1.27)
+				)
+				(hide yes)
+			)
+		)
+		(property "Description" "Generic connector, single row, 01x02, script generated (kicad-library-utils/schlib/autogen/connector/)"
+			(at 172.72 76.2 0)
+			(effects
+				(font
+					(size 1.27 1.27)
+				)
+				(hide yes)
+			)
+		)
+		(pin "2"
+		)
+		(pin "1"
+		)
+		(instances
+			(project ""
+				(path "/bfd666b6-a268-42c4-a4e5-052a7c5965f6"
+					(reference "J103")
+					(unit 1)
+				)
