File: com4bbb.kicad_sch (KiCad schematic)
At the start: 55 parts, among them J101 RS485, J102 PWR, J103 DCF77, J104 PPS, P8 BeagleBone_Black_Header, P9 BeagleBone_Black_Header, SW101 Reset, SW102 PWR, U101 SP3485EN, U102 R-78K5.0-0.5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

Commit message: Add PPS output
Signed-off-by: Benedikt Spranger <b.spranger@linutronix.de>
Parts:
- added J105: PPSOUT, Connector_PinHeader_2.54mm:PinHeader_1x02_P2.54mm_Vertical, symbol Connector_Generic:Conn_01x02
- added Q101: AO3400A, Package_TO_SOT_SMD:SOT-23, symbol Transistor_FET:AO3400A
- added R119: 100, Resistor_SMD:R_0402_1005Metric, symbol Device:R
- added R120: 47k, Resistor_SMD:R_0402_1005Metric, symbol Device:R
- added R121: 1k, Resistor_SMD:R_0402_1005Metric, symbol Device:R
Connections:
- net +5V: now also R121.1
- net GNDD: now also J105.2 (Pin_2), Q101.2 (S), R120.2
- net PPS_OUT: now reaches P9.42 (Pin_42)
- net PPS_OUT: now also R119.1
- new net: J105.1 (Pin_1), Q101.3 (D), R121.2
- new net: Q101.1 (G), R119.2, R120.1
- no-connect marks 43 -> 42
